File: project/Sensors.kicad_sch (KiCad schematic)
At the start: 21 parts, among them IC201 APDS-9306-065, IC202 BMI270, IC203 BMP581, IC204 LIS2MDLTR, IC205 BME688, Q201 DMG1013UW-7

Commit message: Add KiCost
Parts:
- C201, C202, C203, C204, C206, C207, C210, C211, C212: Distributor Mouser -> (none); Mfr. KYOCERA AVX -> (none); Mfr. No. 06035C104KAT2A -> (none); Order No. 581-06035C104KAT2A -> (none); manf (none) -> KYOCERA AVX; manf# (none) -> 06035C104KAT2A; mouser# (none) -> 581-06035C104KAT2A
- C208: Distributor Mouser -> (none); Mfr. KYOCERA AVX -> (none); Mfr. No. 06033C224KAT2A -> (none); Order No. 581-06033C224KAT2A -> (none); manf (none) -> KYOCERA AVX; manf# (none) -> 06033C224KAT2A; mouser# (none) -> 581-06033C224KAT2A
- C209: Distributor Mouser -> (none); Mfr. KYOCERA AVX -> (none); Mfr. No. CM105X5R106M25AT -> (none); Order No. 346-CM105X5R106M25AT -> (none); manf (none) -> KYOCERA AVX; manf# (none) -> CM105X5R106M25AT; mouser# (none) -> 346-CM105X5R106M25AT
- IC201: Distributor Mouser -> (none); Mfr. Broadcom / Avago -> (none); Mfr. No. APDS-9306-065 -> (none); Order No. 630-APDS-9306-065 -> (none); manf (none) -> Broadcom / Avago; manf# (none) -> APDS-9306-065; mouser# (none) -> 630-APDS-9306-065
- IC202: Distributor Mouser -> (none); Mfr. Bosch -> (none); Mfr. No. BMI270 -> (none); Order No. 262-BMI270 -> (none); manf (none) -> Bosch; manf# (none) -> BMI270; mouser# (none) -> 262-BMI270
- IC203: Distributor Mouser -> (none); Mfr. Bosch -> (none); Mfr. No. BMP581 -> (none); Order No. 262-BMP581 -> (none); manf (none) -> Bosch; manf# (none) -> BMP581; mouser# (none) -> 262-BMP581
- IC204: Distributor Mouser -> (none); Mfr. STMicroelectronics -> (none); Mfr. No. LIS2MDLTR -> (none); Order No. 511-LIS2MDLTR -> (none); manf (none) -> STMicroelectronics; manf# (none) -> LIS2MDLTR; mouser# (none) -> 511-LIS2MDLTR
- IC205: Distributor Mouser -> (none); Mfr. Bosch -> (none); Mfr. No. BME688 -> (none); Order No. 262-BME688 -> (none); manf (none) -> Bosch; manf# (none) -> BME688; mouser# (none) -> 262-BME688
- MK201: Distributor Mouser -> (none); Mfr. Knowles -> (none); Mfr. No. SPK0641HT4H-1 -> (none); Order No. 721-SPK0641HT4H-1 -> (none); manf (none) -> Knowles; manf# (none) -> SPK0641HT4H-1; mouser# (none) -> 721-SPK0641HT4H-1
- Q201: Distributor Mouser -> (none); Mfr. Diodes Incorporated -> (none); Mfr. No. DMG1013UW-7 -> (none); Order No. 621-DMG1013UW-7 -> (none); manf (none) -> Diodes Incorporated; manf# (none) -> DMG1013UW-7; mouser# (none) -> 621-DMG1013UW-7
- R201: Distributor Mouser -> (none); Mfr. YAGEO -> (none); Mfr. No. RC0603FR-07150KL -> (none); Order No. 603-RC0603FR-07150KL -> (none); manf (none) -> YAGEO; manf# (none) -> RC0603FR-07150KL; mouser# (none) -> 603-RC0603FR-07150KL
