File: project/Power.kicad_sch (KiCad schematic)
At the start: 20 parts, among them IC101 nPM1300-QEXX, X101 BATTERY

Commit message: Add KiCost
Parts:
- C101, C110: Distributor Mouser -> (none); Mfr. KYOCERA AVX -> (none); Mfr. No. 0603YC105JAT2A -> (none); Order No. 581-0603YC105JAT2A -> (none); manf (none) -> KYOCERA AVX; manf# (none) -> 0603YC105JAT2A; mouser# (none) -> 581-0603YC105JAT2A
- C102: Distributor Mouser -> (none); Mfr. KYOCERA AVX -> (none); Mfr. No. 06035C104KAT2A -> (none); Order No. 581-06035C104KAT2A -> (none); manf (none) -> KYOCERA AVX; manf# (none) -> 06035C104KAT2A; mouser# (none) -> 581-06035C104KAT2A
- C103: Distributor Mouser -> (none); Mfr. KYOCERA AVX -> (none); Mfr. No. 06036D225KAT2A -> (none); Order No. 581-06036D225KAT2A -> (none); manf (none) -> KYOCERA AVX; manf# (none) -> 06036D225KAT2A; mouser# (none) -> 581-06036D225KAT2A
- C104, C105, C106, C107, C108, C109: Distributor Mouser -> (none); Mfr. KYOCERA AVX -> (none); Mfr. No. CM105X5R106M25AT -> (none); Order No. 346-CM105X5R106M25AT -> (none); manf (none) -> KYOCERA AVX; manf# (none) -> CM105X5R106M25AT; mouser# (none) -> 346-CM105X5R106M25AT
- IC101: Distributor Mouser -> (none); Mfr. Nordic Semiconductor -> (none); Mfr. No. nPM1300-QEAA-R7 -> (none); Order No. 949-NPM1300-QEAA-R7 -> (none); manf (none) -> Nordic Semiconductor; manf# (none) -> nPM1300-QEAA-R7; mouser# (none) -> 949-NPM1300-QEAA-R7
- L101, L102: Distributor Mouser -> (none); Mfr. Samsung Electro-Mechanics -> (none); Mfr. No. CIGT201610EH2R2MNE -> (none); Order No. 187-CIGT201610EH2R2MNE -> (none); manf (none) -> Samsung Electro-Mechanics; manf# (none) -> CIGT201610EH2R2MNE; mouser# (none) -> 187-CIGT201610EH2R2MNE
- R101: Distributor Mouser -> (none); Mfr. YAGEO -> (none); Mfr. No. RC0603FR-0747KL -> (none); Order No. 603-RC0603FR-0747KL -> (none); manf (none) -> YAGEO; manf# (none) -> RC0603FR-0747KL; mouser# (none) -> 603-RC0603FR-0747KL
- R102: Distributor Mouser -> (none); Mfr. YAGEO -> (none); Mfr. No. RC0603FR-07150KL -> (none); Order No. 603-RC0603FR-07150KL -> (none); manf (none) -> YAGEO; manf# (none) -> RC0603FR-07150KL; mouser# (none) -> 603-RC0603FR-07150KL
- R103: Distributor Mouser -> (none); Mfr. Bourns -> (none); Mfr. No. CR0402-J/-000GLF -> (none); Order No. 652-CR0603-J/-000ELF -> (none); manf (none) -> Bourns; manf# (none) -> CR0402-J/-000GLF; mouser# (none) -> 652-CR0603-J/-000ELF
- X101: Distributor Mouser -> (none); Mfr. Molex -> (none); Mfr. No. 78171-0002 -> (none); Order No. 538-78171-0002 -> (none); manf (none) -> Molex; manf# (none) -> 78171-0002; mouser# (none) -> 538-78171-0002

Commit message: Fix wrong part numbers
Parts:
- C103: mouser# 581-06036D225KAT2A -> 581-06036D225K
- L101, L102: mouser# 187-CIGT201610EH2R2MNE -> 187-CIGT201610EH2R2M
Changed lines of the file:
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@@
 			)
 		)
-		(property "mouser#" "187-CIGT201610EH2R2MNE"
+		(property "mouser#" "187-CIGT201610EH2R2M"
 			(at 173.99 106.68 0)
 			(effects
@@
 			)
 		)
-		(property "mouser#" "187-CIGT201610EH2R2MNE"
+		(property "mouser#" "187-CIGT201610EH2R2M"
 			(at 182.88 88.9 0)
 			(effects
@@
 			)
 		)
-		(property "mouser#" "581-06036D225KAT2A"
+		(property "mouser#" "581-06036D225K"
 			(at 140.97 44.45 0)
 			(effects

Commit message: Rebase with upstream 2.0.6
Parts:
- L101, L102: manf Samsung Electro-Mechanics -> Vishay / Dale; manf# CIGT201610EH2R2MNE -> IHLL0806AZEZ2R2M1Z; mouser# 187-CIGT201610EH2R2M -> 70-IHLL0806AZZ2R2M1Z
Changed lines of the file:
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@@
 			)
 		)
-		(property "Datasheet" "https://www.mouser.de/datasheet/2/585/sems_s_a0006918008_1-2288745.pdf"
+		(property "Datasheet" "https://www.vishay.com/doc?34649"
 			(at 173.99 106.68 0)
 			(effects
@@
 			)
 		)
-		(property "manf" "Samsung Electro-Mechanics"
+		(property "manf" "Vishay / Dale"
 			(at 173.99 106.68 0)
 			(effects
@@
 			)
 		)
-		(property "manf#" "CIGT201610EH2R2MNE"
+		(property "manf#" "IHLL0806AZEZ2R2M1Z"
 			(at 173.99 106.68 0)
 			(effects
@@
 			)
 		)
-		(property "mouser#" "187-CIGT201610EH2R2M"
+		(property "mouser#" "70-IHLL0806AZZ2R2M1Z"
 			(at 173.99 106.68 0)
 			(effects
@@
 			)
 		)
-		(property "Datasheet" "https://www.mouser.de/datasheet/2/585/sems_s_a0006918008_1-2288745.pdf"
+		(property "Datasheet" "https://www.vishay.com/doc?34649"
 			(at 182.88 88.9 0)
 			(effects
@@
 			)
 		)
-		(property "manf" "Samsung Electro-Mechanics"
+		(property "manf" "Vishay / Dale"
 			(at 182.88 88.9 0)
 			(effects
@@
 			)
 		)
-		(property "manf#" "CIGT201610EH2R2MNE"
+		(property "manf#" "IHLL0806AZEZ2R2M1Z"
 			(at 182.88 88.9 0)
 			(effects
@@
 			)
 		)
-		(property "mouser#" "187-CIGT201610EH2R2M"
+		(property "mouser#" "70-IHLL0806AZZ2R2M1Z"
 			(at 182.88 88.9 0)
 			(effects
