File: watch/MCU.kicad_sch (KiCad schematic)
At the start: 14 parts, among them IC601 FAN5622SX, IC602 USBLC6-2P6, IC603 MX25U51245GZ4I00, IC604 NTS0104GU12, M601 NORA-B106, X603 Device, X608 Display

Commit message: OPtimize connector positions
- New position for the battery connector, moved to the right side of the watch
- Rotate haptics connector by 180°
Parts:
- R601: manf (none) -> YAGEO; manf# (none) -> RC0201JR-0712KL; mouser# (none) -> 603-RC0201JR-0712KL
- R612, R613: manf (none) -> YAGEO; manf# (none) -> RC0201JR-07100KL; mouser# (none) -> 603-RC0201JR-07100KL
Changed lines of the file:
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@@
 			)
 		)
-		(property "Datasheet" ""
+		(property "Datasheet" "https://www.mouser.com/catalog/specsheets/YAGEO_PYu_RC_Group_51_RoHS_L_12.pdf"
 			(at 215.9 185.42 0)
 			(effects
@@
 			)
 		)
-		(property "manf" ""
+		(property "manf" "YAGEO"
 			(at 215.9 185.42 0)
 			(effects
@@
 			)
 		)
-		(property "manf#" ""
+		(property "manf#" "RC0201JR-07100KL"
 			(at 215.9 185.42 0)
 			(effects
@@
 			)
 		)
-		(property "mouser#" ""
+		(property "mouser#" "603-RC0201JR-07100KL"
 			(at 215.9 185.42 0)
 			(effects
@@
 			)
 		)
-		(property "Datasheet" ""
+		(property "Datasheet" "https://www.mouser.com/catalog/specsheets/YAGEO_PYu_RC_Group_51_RoHS_L_12.pdf"
 			(at 331.47 60.96 0)
 			(effects
@@
 			)
 		)
-		(property "manf" ""
+		(property "manf" "YAGEO"
 			(at 331.47 60.96 0)
 			(effects
@@
 			)
 		)
-		(property "manf#" ""
+		(property "manf#" "RC0201JR-07100KL"
 			(at 331.47 60.96 0)
 			(effects
@@
 			)
 		)
-		(property "mouser#" ""
+		(property "mouser#" "603-RC0201JR-07100KL"
 			(at 331.47 60.96 0)
 			(effects
@@
 			)
 		)
-		(property "Datasheet" ""
+		(property "Datasheet" "https://www.mouser.com/catalog/specsheets/YAGEO_PYu_RC_Group_51_RoHS_L_12.pdf"
 			(at 36.83 199.39 0)
 			(effects
@@
 			)
 		)
-		(property "manf" ""
+		(property "manf" "YAGEO"
 			(at 36.83 199.39 0)
 			(effects
@@
 			)
 		)
-		(property "manf#" ""
+		(property "manf#" "RC0201JR-0712KL"
 			(at 36.83 199.39 0)
 			(effects
@@
 			)
 		)
-		(property "mouser#" ""
+		(property "mouser#" "603-RC0201JR-0712KL"
 			(at 36.83 199.39 0)
 			(effects
