File: watch/MCU.kicad_sch (KiCad schematic)
At the start: 16 parts, among them IC601 FAN5622SX, IC602 USBLC6-2P6, IC603 MX25U51245GZ4I00, IC604 NTS0104GU12, M601 NORA-B106, X603 Device, X608 Display

Commit message: Update schematic and layout with KiCad 10
Changes to the MCU and Power sheets and the layout, saved with KiCad 10
(adds the new KiCad 10 project settings).

Co-Authored-By: Claude Opus 5.5 <noreply@anthropic.com>
Parts:
- TP7, TP8: footprint TestPoint:TestPoint_Pad_D1.0mm -> Testpoints_Kampi:TestPoint_Pad_D1.0mm; now left out of the parts list
Other:
- moved on the sheet: TP7, TP8
Changed lines of the file:
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@@
 	(wire
 		(pts
-			(xy 231.14 121.92) (xy 257.81 121.92)
+			(xy 231.14 121.92) (xy 259.08 121.92)
 		)
 		(stroke
@@
 	(wire
 		(pts
-			(xy 257.81 121.92) (xy 257.81 119.38)
+			(xy 259.08 121.92) (xy 259.08 118.11)
 		)
 		(stroke
@@
 	(wire
 		(pts
-			(xy 231.14 119.38) (xy 247.65 119.38)
-		)
-		(stroke
-			(width 0)
-			(type default)
-		)
-	)
-	(wire
-		(pts
 			(xy 237.49 175.26) (xy 240.03 175.26)
 		)
@@
 	(wire
 		(pts
+			(xy 247.65 119.38) (xy 231.14 119.38)
+		)
+		(stroke
+			(width 0)
+			(type default)
+		)
+	)
+	(wire
+		(pts
 			(xy 109.22 96.52) (xy 107.95 96.52)
 		)
@@
 	(wire
 		(pts
+			(xy 247.65 118.11) (xy 247.65 119.38)
+		)
+		(stroke
+			(width 0)
+			(type default)
+		)
+	)
+	(wire
+		(pts
 			(xy 109.22 224.79) (xy 110.49 224.79)
 		)
@@
 	(symbol
 		(lib_id "Connector:TestPoint")
-		(at 247.65 119.38 0)
+		(at 247.65 118.11 0)
 		(unit 1)
 		(body_style 1)
 		(exclude_from_sim no)
-		(in_bom yes)
+		(in_bom no)
 		(on_board yes)
-		(in_pos_files yes)
+		(in_pos_files no)
 		(dnp no)
+		(fields_autoplaced yes)
 		(property "Reference" "TP7"
-			(at 244.094 110.744 0)
+			(at 247.65 109.22 0)
 			(show_name no)
 			(do_not_autoplace no)
@@
 					(size 1.27 1.27)
 				)
-				(justify left)
 			)
 		)
 		(property "Value" "TestPoint"
-			(at 242.57 112.268 0)
+			(at 247.65 111.76 0)
 			(show_name no)
 			(do_not_autoplace no)
@@
 					(size 1.27 1.27)
 				)
-				(justify left)
 			)
 		)
-		(property "Footprint" "TestPoint:TestPoint_Pad_D1.0mm"
-			(at 252.73 119.38 0)
+		(property "Footprint" "Testpoints_Kampi:TestPoint_Pad_D1.0mm"
+			(at 252.73 118.11 0)
 			(hide yes)
 			(show_name no)
@@
 		)
 		(property "Datasheet" ""
-			(at 252.73 119.38 0)
+			(at 252.73 118.11 0)
 			(hide yes)
 			(show_name no)
@@
 		)
 		(property "Description" "test point"
-			(at 247.65 119.38 0)
+			(at 247.65 118.11 0)
+			(hide yes)
+			(show_name no)
+			(do_not_autoplace no)
+			(effects
+				(font
+					(size 1.27 1.27)
+				)
+			)
+		)
+		(property "manf" ""
+			(at 247.65 118.11 0)
+			(hide yes)
+			(show_name no)
+			(do_not_autoplace no)
+			(effects
+				(font
+					(size 1.27 1.27)
+				)
+			)
+		)
+		(property "manf#" ""
+			(at 247.65 118.11 0)
+			(hide yes)
+			(show_name no)
+			(do_not_autoplace no)
+			(effects
+				(font
+					(size 1.27 1.27)
+				)
+			)
+		)
+		(property "mouser#" ""
+			(at 247.65 118.11 0)
+			(hide yes)
+			(show_name no)
+			(do_not_autoplace no)
+			(effects
+				(font
+					(size 1.27 1.27)
+				)
+			)
+		)
+		(property "Config" ""
+			(at 247.65 118.11 0)
 			(hide yes)
 			(show_name no)
@@
 	(symbol
 		(lib_id "Connector:TestPoint")
-		(at 257.81 119.38 0)
+		(at 259.08 118.11 0)
 		(unit 1)
 		(body_style 1)
 		(exclude_from_sim no)
-		(in_bom yes)
+		(in_bom no)
 		(on_board yes)
-		(in_pos_files yes)
+		(in_pos_files no)
 		(dnp no)
+		(fields_autoplaced yes)
 		(property "Reference" "TP8"
-			(at 254.254 110.744 0)
+			(at 261.62 113.5379 0)
 			(show_name no)
 			(do_not_autoplace no)
@@
 		)
 		(property "Value" "TestPoint"
-			(at 252.73 112.268 0)
+			(at 261.62 116.0779 0)
 			(show_name no)
 			(do_not_autoplace no)
@@
 			)
 		)
-		(property "Footprint" "TestPoint:TestPoint_Pad_D1.0mm"
-			(at 262.89 119.38 0)
+		(property "Footprint" "Testpoints_Kampi:TestPoint_Pad_D1.0mm"
+			(at 264.16 118.11 0)
 			(hide yes)
 			(show_name no)
@@
 		)
 		(property "Datasheet" ""
-			(at 262.89 119.38 0)
+			(at 264.16 118.11 0)
 			(hide yes)
 			(show_name no)
@@
 		)
 		(property "Description" "test point"
-			(at 257.81 119.38 0)
+			(at 259.08 118.11 0)
+			(hide yes)
+			(show_name no)
+			(do_not_autoplace no)
+			(effects
+				(font
+					(size 1.27 1.27)
+				)
+			)
+		)
+		(property "manf" ""
+			(at 259.08 118.11 0)
+			(hide yes)
+			(show_name no)
+			(do_not_autoplace no)
+			(effects
+				(font
+					(size 1.27 1.27)
+				)
+			)
+		)
+		(property "manf#" ""
+			(at 259.08 118.11 0)
+			(hide yes)
+			(show_name no)
+			(do_not_autoplace no)
+			(effects
+				(font
+					(size 1.27 1.27)
+				)
+			)
+		)
+		(property "mouser#" ""
+			(at 259.08 118.11 0)
+			(hide yes)
+			(show_name no)
+			(do_not_autoplace no)
+			(effects
+				(font
+					(size 1.27 1.27)
+				)
+			)
+		)
+		(property "Config" ""
+			(at 259.08 118.11 0)
 			(hide yes)
 			(show_name no)
