File: watch/Peripherals.kicad_sch (KiCad schematic)
At the start: 30 parts, among them IC501 APDS-9306-065, IC502 BMI270, IC503 LIS2MDLTR, IC504 BMP581, IC505 DRV2603RUNT, IC506 PCA9306JK, IC507 RV-8263-C8, M501 Vibrator DC Motor, X509 Motor

Commit message: New buttons
Signed-off-by: Daniel Kampert <DanielKampert@kampis-elektroecke.de>
Parts:
- S501, S502, S503, S504: footprint E-Switch:TL6340AF160Q_Modified -> Wuerth:43633303381_NoMountingPads; manf E-Switch -> Wurth Elektronik; manf# TL6340AF160Q -> 436333033816; mouser# 612-TL6340AF160Q -> 710-436333033816
Connections:
- net GND: now also S501.1, S504.1; no longer S501.2, S504.2
- net SW1: now also S501.2; no longer S501.1
- net SW4: now also S504.2; no longer S504.1
Changed lines of the file:
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@@
 			)
 		)
-		(property "Footprint" "E-Switch:TL6340AF160Q_Modified"
+		(property "Footprint" "Wuerth:43633303381_NoMountingPads"
 			(at 25.4 118.11 0)
 			(effects
@@
 			)
 		)
-		(property "Datasheet" "https://www.mouser.de/datasheet/2/140/TL6340-3304863.pdf"
+		(property "Datasheet" "https://www.we-online.com/components/products/datasheet/436333033816.pdf"
 			(at 25.4 118.11 0)
 			(effects
@@
 			)
 		)
-		(property "manf" "E-Switch"
+		(property "manf" "Wurth Elektronik"
 			(at 25.4 123.19 0)
 			(effects
@@
 			)
 		)
-		(property "manf#" "TL6340AF160Q"
+		(property "manf#" "436333033816"
 			(at 25.4 123.19 0)
 			(effects
@@
 			)
 		)
-		(property "mouser#" "612-TL6340AF160Q"
+		(property "mouser#" "710-436333033816"
 			(at 25.4 123.19 0)
 			(effects
@@
 		(lib_id "Switch:SW_Push")
 		(at 25.4 134.62 0)
-		(mirror y)
 		(unit 1)
 		(exclude_from_sim no)
@@
 		(on_board yes)
 		(dnp no)
-		(fields_autoplaced yes)
 		(property "Reference" "S504"
 			(at 25.4 127 0)
@@
 			)
 		)
-		(property "Footprint" "E-Switch:TL6340AF160Q_Modified"
+		(property "Footprint" "Wuerth:43633303381_NoMountingPads"
 			(at 25.4 129.54 0)
 			(effects
@@
 			)
 		)
-		(property "Datasheet" "https://www.mouser.de/datasheet/2/140/TL6340-3304863.pdf"
+		(property "Datasheet" "https://www.we-online.com/components/products/datasheet/436333033816.pdf"
 			(at 25.4 129.54 0)
 			(effects
@@
 			)
 		)
-		(property "manf" "E-Switch"
+		(property "manf" "Wurth Elektronik"
 			(at 25.4 134.62 0)
 			(effects
@@
 			)
 		)
-		(property "manf#" "TL6340AF160Q"
+		(property "manf#" "436333033816"
 			(at 25.4 134.62 0)
 			(effects
@@
 			)
 		)
-		(property "mouser#" "612-TL6340AF160Q"
+		(property "mouser#" "710-436333033816"
 			(at 25.4 134.62 0)
 			(effects
@@
 		(lib_id "Switch:SW_Push")
 		(at 25.4 100.33 0)
-		(mirror y)
 		(unit 1)
 		(exclude_from_sim no)
@@
 		(on_board yes)
 		(dnp no)
-		(fields_autoplaced yes)
 		(property "Reference" "S501"
 			(at 25.4 92.71 0)
@@
 			)
 		)
-		(property "Footprint" "E-Switch:TL6340AF160Q_Modified"
+		(property "Footprint" "Wuerth:43633303381_NoMountingPads"
 			(at 25.4 95.25 0)
 			(effects
@@
 			)
 		)
-		(property "Datasheet" "https://www.mouser.de/datasheet/2/140/TL6340-3304863.pdf"
+		(property "Datasheet" "https://www.we-online.com/components/products/datasheet/436333033816.pdf"
 			(at 25.4 95.25 0)
 			(effects
@@
 			)
 		)
-		(property "manf" "E-Switch"
+		(property "manf" "Wurth Elektronik"
 			(at 25.4 100.33 0)
 			(effects
@@
 			)
 		)
-		(property "manf#" "TL6340AF160Q"
+		(property "manf#" "436333033816"
 			(at 25.4 100.33 0)
 			(effects
@@
 			)
 		)
-		(property "mouser#" "612-TL6340AF160Q"
+		(property "mouser#" "710-436333033816"
 			(at 25.4 100.33 0)
 			(effects
@@
 			)
 		)
-		(property "Footprint" "E-Switch:TL6340AF160Q_Modified"
+		(property "Footprint" "Wuerth:43633303381_NoMountingPads"
 			(at 25.4 106.68 0)
 			(effects
@@
 			)
 		)
-		(property "Datasheet" "https://www.mouser.de/datasheet/2/140/TL6340-3304863.pdf"
+		(property "Datasheet" "https://www.we-online.com/components/products/datasheet/436333033816.pdf"
 			(at 25.4 106.68 0)
 			(effects
@@
 			)
 		)
-		(property "manf" "E-Switch"
+		(property "manf" "Wurth Elektronik"
 			(at 25.4 111.76 0)
 			(effects
@@
 			)
 		)
-		(property "manf#" "TL6340AF160Q"
+		(property "manf#" "436333033816"
 			(at 25.4 111.76 0)
 			(effects
@@
 			)
 		)
-		(property "mouser#" "612-TL6340AF160Q"
+		(property "mouser#" "710-436333033816"
 			(at 25.4 111.76 0)
 			(effects

Commit message: OPtimize connector positions
- New position for the battery connector, moved to the right side of the watch
- Rotate haptics connector by 180°
Parts:
- C505: manf (none) -> KYOCERA AVX; manf# (none) -> 0201ZD224KAT2A; mouser# (none) -> 581-0201ZD224KAT2A
- MK501: manf# (none) -> SPK0641HT4H-1; mouser# (none) -> 721-SPK0641HT4H-1
- R501, R502: manf (none) -> YAGEO; manf# (none) -> RC0201JR-071K8L; mouser# (none) -> 603-RC0201JR-071K8L
- R504, R505: manf (none) -> YAGEO; manf# (none) -> RC0201JR-073K3L; mouser# (none) -> 603-RC0201JR-073K3L
- R506: manf (none) -> YAGEO; manf# (none) -> RC0201JR-07200KL; mouser# (none) -> 603-RC0201JR-07200KL
Changed lines of the file:
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@@
 			)
 		)
-		(property "Datasheet" ""
+		(property "Datasheet" "https://www.mouser.com/catalog/specsheets/YAGEO_PYu_RC_Group_51_RoHS_L_12.pdf"
 			(at 353.06 107.95 0)
 			(effects
@@
 			)
 		)
-		(property "manf" ""
+		(property "manf" "YAGEO"
 			(at 353.06 107.95 0)
 			(effects
@@
 			)
 		)
-		(property "manf#" ""
+		(property "manf#" "RC0201JR-07200KL"
 			(at 353.06 107.95 0)
 			(effects
@@
 			)
 		)
-		(property "mouser#" ""
+		(property "mouser#" "603-RC0201JR-07200KL"
 			(at 353.06 107.95 0)
 			(effects
@@
 			)
 		)
-		(property "Datasheet" ""
+		(property "Datasheet" "https://www.mouser.com/catalog/specsheets/YAGEO_PYu_RC_Group_51_RoHS_L_12.pdf"
 			(at 364.49 121.92 0)
 			(effects
@@
 			)
 		)
-		(property "manf" ""
+		(property "manf" "YAGEO"
 			(at 364.49 121.92 0)
 			(effects
@@
 			)
 		)
-		(property "manf#" ""
+		(property "manf#" "RC0201JR-073K3L"
 			(at 364.49 121.92 0)
 			(effects
@@
 			)
 		)
-		(property "mouser#" ""
+		(property "mouser#" "603-RC0201JR-073K3L"
 			(at 364.49 121.92 0)
 			(effects
@@
 			)
 		)
-		(property "Datasheet" "~"
+		(property "Datasheet" "https://www.vybronics.com/wp-content/uploads/datasheet-files/Vybronics-VC1027B902F-Jinlong-C1027B902F-datasheet.pdf"
 			(at 379.73 61.976 0)
 			(effects
@@
 			)
 		)
-		(property "Datasheet" ""
+		(property "Datasheet" "https://datasheets.kyocera-avx.com/cx5r-KGM.pdf"
 			(at 240.03 166.37 0)
 			(effects
@@
 			)
 		)
-		(property "manf" ""
+		(property "manf" "KYOCERA AVX"
 			(at 240.03 166.37 0)
 			(effects
@@
 			)
 		)
-		(property "manf#" ""
+		(property "manf#" "0201ZD224KAT2A"
 			(at 240.03 166.37 0)
 			(effects
@@
 			)
 		)
-		(property "mouser#" ""
+		(property "mouser#" "581-0201ZD224KAT2A"
 			(at 240.03 166.37 0)
 			(effects
@@
 			)
 		)
-		(property "Datasheet" ""
+		(property "Datasheet" "https://www.mouser.com/catalog/specsheets/YAGEO_PYu_RC_Group_51_RoHS_L_12.pdf"
 			(at 314.96 121.92 0)
 			(effects
@@
 			)
 		)
-		(property "manf" ""
+		(property "manf" "YAGEO"
 			(at 314.96 121.92 0)
 			(effects
@@
 			)
 		)
-		(property "manf#" ""
+		(property "manf#" "RC0201JR-071K8L"
 			(at 314.96 121.92 0)
 			(effects
@@
 			)
 		)
-		(property "mouser#" ""
+		(property "mouser#" "603-RC0201JR-071K8L"
 			(at 314.96 121.92 0)
 			(effects
@@
 			)
 		)
-		(property "Datasheet" ""
+		(property "Datasheet" "https://www.mouser.com/catalog/specsheets/YAGEO_PYu_RC_Group_51_RoHS_L_12.pdf"
 			(at 367.03 121.92 0)
 			(effects
@@
 			)
 		)
-		(property "manf" ""
+		(property "manf" "YAGEO"
 			(at 367.03 121.92 0)
 			(effects
@@
 			)
 		)
-		(property "manf#" ""
+		(property "manf#" "RC0201JR-073K3L"
 			(at 367.03 121.92 0)
 			(effects
@@
 			)
 		)
-		(property "mouser#" ""
+		(property "mouser#" "603-RC0201JR-073K3L"
 			(at 367.03 121.92 0)
 			(effects
@@
 			)
 		)
-		(property "manf#" ""
+		(property "manf#" "SPK0641HT4H-1"
 			(at 86.36 127 0)
 			(effects
@@
 			)
 		)
-		(property "mouser#" ""
+		(property "mouser#" "721-SPK0641HT4H-1"
 			(at 86.36 127 0)
 			(effects
@@
 			)
 		)
-		(property "Datasheet" ""
+		(property "Datasheet" "https://www.mouser.com/catalog/specsheets/YAGEO_PYu_RC_Group_51_RoHS_L_12.pdf"
 			(at 312.42 121.92 0)
 			(effects
@@
 			)
 		)
-		(property "manf" ""
+		(property "manf" "YAGEO"
 			(at 312.42 121.92 0)
 			(effects
@@
 			)
 		)
-		(property "manf#" ""
+		(property "manf#" "RC0201JR-071K8L"
 			(at 312.42 121.92 0)
 			(effects
@@
 			)
 		)
-		(property "mouser#" ""
+		(property "mouser#" "603-RC0201JR-071K8L"
 			(at 312.42 121.92 0)
 			(effects
