File: watch/Power.kicad_sch (KiCad schematic)
At the start: 17 parts, among them IC401 nPM1300-QEXX, X402 Battery

Commit message: New battery connector
- Add CI/CD workflow to check for changelog updates on pull requests

Signed-off-by: Daniel Kampert <DanielKampert|kampis-elektroecke.de>
Parts:
- X402: footprint Molex:78171-0002 -> JST_SH_SM02B-SRSS-TB_1x02-1MP_P1.00mm_Horizontal; manf Molex -> (none); manf# 78171-0002 -> (none); mouser# 538-78171-0002 -> (none)
Changed lines of the file:
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@@
 			)
 		)
-		(property "Footprint" "Molex:78171-0002"
+		(property "Footprint" "JST_SH_SM02B-SRSS-TB_1x02-1MP_P1.00mm_Horizontal"
 			(at 198.12 36.83 0)
 			(effects
@@
 			)
 		)
-		(property "Datasheet" "https://www.molex.com/en-us/products/part-detail-pdf/781710002?display=pdf"
+		(property "Datasheet" ""
 			(at 198.12 36.83 0)
 			(effects
@@
 			)
 		)
-		(property "manf" "Molex"
+		(property "manf" ""
 			(at 198.12 36.83 0)
 			(effects
@@
 			)
 		)
-		(property "manf#" "78171-0002"
+		(property "manf#" ""
 			(at 198.12 36.83 0)
 			(effects
@@
 			)
 		)
-		(property "mouser#" "538-78171-0002"
+		(property "mouser#" ""
 			(at 198.12 36.83 0)
 			(effects

Commit message: OPtimize connector positions
- New position for the battery connector, moved to the right side of the watch
- Rotate haptics connector by 180°
Parts:
- R407: manf (none) -> YAGEO; manf# (none) -> RC0201JR-0747KL; mouser# (none) -> 603-RC0201JR-0747KL
- R408: manf (none) -> YAGEO; manf# (none) -> RC0201JR-07100KL; mouser# (none) -> 603-RC0201JR-07100KL
Changed lines of the file:
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@@
 			)
 		)
-		(property "Datasheet" ""
+		(property "Datasheet" "https://www.mouser.com/catalog/specsheets/YAGEO_PYu_RC_Group_51_RoHS_L_12.pdf"
 			(at 120.65 130.81 0)
 			(effects
@@
 			)
 		)
-		(property "manf" ""
+		(property "manf" "YAGEO"
 			(at 120.65 130.81 0)
 			(effects
@@
 			)
 		)
-		(property "manf#" ""
+		(property "manf#" "RC0201JR-07100KL"
 			(at 120.65 130.81 0)
 			(effects
@@
 			)
 		)
-		(property "mouser#" ""
+		(property "mouser#" "603-RC0201JR-07100KL"
 			(at 120.65 130.81 0)
 			(effects
@@
 			)
 		)
-		(property "manf" ""
+		(property "manf" "YAGEO"
 			(at 118.11 130.81 0)
 			(effects
@@
 			)
 		)
-		(property "manf#" ""
+		(property "manf#" "RC0201JR-0747KL"
 			(at 118.11 130.81 0)
 			(effects
@@
 			)
 		)
-		(property "mouser#" ""
+		(property "mouser#" "603-RC0201JR-0747KL"
 			(at 118.11 130.81 0)
 			(effects

Commit message: Rename PCB workflow, add part number for battery connector, remove sim pins property
Parts:
- X402: manf (none) -> JST Commercial; manf# (none) -> SM02B-SRSS-TB; mouser# (none) -> 306-SM02BSRSSTBLFSN
Changed lines of the file:
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@@
 			)
 		)
-		(property "Sim.Pins" ""
-			(at 220.98 50.8 0)
-			(effects
-				(font
-					(size 1.27 1.27)
-				)
-				(hide yes)
-			)
-		)
 		(pin "1"
 		)
@@
 			)
 		)
-		(property "Sim.Pins" ""
-			(at 212.09 102.87 0)
-			(effects
-				(font
-					(size 1.27 1.27)
-				)
-				(hide yes)
-			)
-		)
 		(pin "1"
 		)
@@
 			)
 		)
-		(property "Sim.Pins" ""
-			(at 143.51 46.99 0)
-			(effects
-				(font
-					(size 1.27 1.27)
-				)
-				(hide yes)
-			)
-		)
 		(pin "1"
 		)
@@
 			)
 		)
-		(property "Sim.Pins" ""
-			(at 222.25 105.41 0)
-			(effects
-				(font
-					(size 1.27 1.27)
-				)
-				(hide yes)
-			)
-		)
 		(pin "1"
 		)
@@
 			)
 		)
-		(property "Sim.Pins" ""
-			(at 120.65 130.81 0)
-			(effects
-				(font
-					(size 1.27 1.27)
-				)
-				(hide yes)
-			)
-		)
 		(pin "1"
 		)
@@
 			)
 		)
-		(property "Sim.Pins" ""
-			(at 231.14 87.63 0)
-			(effects
-				(font
-					(size 1.27 1.27)
-				)
-				(hide yes)
-			)
-		)
 		(pin "1"
 		)
@@
 			)
 		)
-		(property "Sim.Pins" ""
-			(at 118.11 130.81 0)
-			(effects
-				(font
-					(size 1.27 1.27)
-				)
-				(hide yes)
-			)
-		)
 		(pin "1"
 		)
@@
 			)
 		)
-		(property "Sim.Pins" ""
-			(at 170.18 104.14 0)
-			(effects
-				(font
-					(size 1.27 1.27)
-				)
-				(hide yes)
-			)
-		)
 		(pin "1"
 		)
@@
 			)
 		)
-		(property "Sim.Pins" ""
-			(at 236.22 33.02 0)
-			(effects
-				(font
-					(size 1.27 1.27)
-				)
-				(hide yes)
-			)
-		)
 		(pin "1"
 		)
@@
 			)
 		)
-		(property "Sim.Pins" ""
-			(at 220.98 85.09 0)
-			(effects
-				(font
-					(size 1.27 1.27)
-				)
-				(hide yes)
-			)
-		)
 		(pin "1"
 		)
@@
 			)
 		)
-		(property "Datasheet" ""
+		(property "Datasheet" "https://www.mouser.com/catalog/specsheets/JST_SM02B-SRSS-TB_LF_SN_eSR_SZ.pdf"
 			(at 198.12 36.83 0)
 			(effects
@@
 			)
 		)
-		(property "manf" ""
-			(at 198.12 36.83 0)
-			(effects
-				(font
-					(size 1.27 1.27)
-				)
-				(hide yes)
-			)
-		)
-		(property "manf#" ""
+		(property "manf" "JST Commercial"
 			(at 198.12 36.83 0)
 			(effects
@@
 			)
 		)
-		(property "mouser#" ""
+		(property "manf#" "SM02B-SRSS-TB"
 			(at 198.12 36.83 0)
 			(effects
@@
 			)
 		)
-		(property "Sim.Pins" ""
+		(property "mouser#" "306-SM02BSRSSTBLFSN"
 			(at 198.12 36.83 0)
 			(effects
@@
 			)
 		)
-		(property "Sim.Pins" ""
-			(at 215.9 137.16 0)
-			(effects
-				(font
-					(size 1.27 1.27)
-				)
-				(hide yes)
-			)
-		)
 		(pin "1"
 		)
@@
 			)
 		)
-		(property "Sim.Pins" ""
-			(at 226.06 33.02 0)
-			(effects
-				(font
-					(size 1.27 1.27)
-				)
-				(hide yes)
-			)
-		)
 		(pin "1"
 		)
@@
 			)
 		)
-		(property "Sim.Pins" ""
-			(at 179.07 40.64 0)
-			(effects
-				(font
-					(size 1.27 1.27)
-				)
-				(hide yes)
-			)
-		)
 		(pin "1"
 		)
@@
 			)
 		)
-		(property "Sim.Pins" ""
-			(at 166.37 40.64 0)
-			(effects
-				(font
-					(size 1.27 1.27)
-				)
-				(hide yes)
-			)
-		)
 		(pin "1"
 		)
@@
 			)
 		)
-		(property "Sim.Pins" ""
-			(at 246.38 33.02 0)
-			(effects
-				(font
-					(size 1.27 1.27)
-				)
-				(hide yes)
-			)
-		)
 		(pin "1"
 		)
@@
 			(at 231.14 133.35 0)
 			(effects
-				(font
-					(size 1.27 1.27)
-				)
-				(hide yes)
-			)
-		)
-		(property "Sim.Pins" ""
-			(at 231.14 133.35 0)
-			(effects
