File: watch/Power.kicad_sch (KiCad schematic)
At the start: 22 parts, among them IC401 nPM1300-QEXX, J1 53261-0271

Commit message: Update schematic and layout with KiCad 10
Changes to the MCU and Power sheets and the layout, saved with KiCad 10
(adds the new KiCad 10 project settings).

Co-Authored-By: Claude Opus 5.5 <noreply@anthropic.com>
Parts:
- TP4, TP5, TP6: footprint TestPoint:TestPoint_Pad_D1.0mm -> Testpoints_Kampi:TestPoint_Pad_D1.0mm; now left out of the parts list
Other:
- moved on the sheet: TP4, TP5, TP6
Changed lines of the file:
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@@
 	)
 	(junction
-		(at 252.73 29.21)
+		(at 231.14 83.82)
 		(diameter 0)
 		(color 0 0 0 0)
 	)
 	(junction
-		(at 231.14 83.82)
+		(at 215.9 130.81)
 		(diameter 0)
 		(color 0 0 0 0)
 	)
 	(junction
-		(at 215.9 130.81)
+		(at 252.73 29.21)
+		(diameter 0)
+		(color 0 0 0 0)
+	)
+	(junction
+		(at 242.57 83.82)
 		(diameter 0)
 		(color 0 0 0 0)
@@
 	)
 	(junction
+		(at 242.57 101.6)
+		(diameter 0)
+		(color 0 0 0 0)
+	)
+	(junction
 		(at 220.98 46.99)
 		(diameter 0)
@@
 	)
 	(junction
-		(at 242.57 83.82)
-		(diameter 0)
-		(color 0 0 0 0)
-	)
-	(junction
 		(at 231.14 123.19)
 		(diameter 0)
@@
 		(color 0 0 0 0)
 	)
-	(junction
-		(at 242.57 101.6)
-		(diameter 0)
-		(color 0 0 0 0)
-	)
 	(no_connect
 		(at 200.66 13.97)
@@
 	(wire
 		(pts
+			(xy 242.57 100.33) (xy 242.57 101.6)
+		)
+		(stroke
+			(width 0)
+			(type default)
+		)
+	)
+	(wire
+		(pts
 			(xy 173.99 36.83) (xy 173.99 66.04)
 		)
@@
 	(wire
 		(pts
+			(xy 252.73 27.94) (xy 252.73 29.21)
+		)
+		(stroke
+			(width 0)
+			(type default)
+		)
+	)
+	(wire
+		(pts
 			(xy 227.33 80.01) (xy 227.33 83.82)
 		)
@@
 	(wire
 		(pts
-			(xy 242.57 83.82) (xy 251.46 83.82)
+			(xy 207.01 109.22) (xy 222.25 109.22)
 		)
 		(stroke
@@
 	(wire
 		(pts
-			(xy 207.01 109.22) (xy 222.25 109.22)
+			(xy 231.14 83.82) (xy 231.14 85.09)
 		)
 		(stroke
@@
 	(wire
 		(pts
-			(xy 231.14 83.82) (xy 231.14 85.09)
+			(xy 242.57 83.82) (xy 251.46 83.82)
+		)
+		(stroke
+			(width 0)
+			(type default)
+		)
+	)
+	(wire
+		(pts
+			(xy 242.57 101.6) (xy 251.46 101.6)
 		)
 		(stroke
@@
 	(wire
 		(pts
-			(xy 242.57 101.6) (xy 251.46 101.6)
-		)
-		(stroke
-			(width 0)
-			(type default)
-		)
-	)
-	(wire
-		(pts
 			(xy 226.06 29.21) (xy 213.36 29.21)
 		)
@@
 	(wire
 		(pts
+			(xy 242.57 82.55) (xy 242.57 83.82)
+		)
+		(stroke
+			(width 0)
+			(type default)
+		)
+	)
+	(wire
+		(pts
 			(xy 226.06 29.21) (xy 226.06 30.48)
 		)
@@
 	(wire
 		(pts
-			(xy 252.73 29.21) (xy 264.16 29.21)
-		)
-		(stroke
-			(width 0)
-			(type default)
-		)
-	)
-	(wire
-		(pts
 			(xy 231.14 121.92) (xy 231.14 123.19)
 		)
@@
 	(wire
 		(pts
+			(xy 252.73 29.21) (xy 264.16 29.21)
+		)
+		(stroke
+			(width 0)
+			(type default)
+		)
+	)
+	(wire
+		(pts
 			(xy 220.98 80.01) (xy 220.98 81.28)
 		)
@@
 	(symbol
 		(lib_id "Connector:TestPoint")
-		(at 252.73 29.21 0)
+		(at 252.73 27.94 0)
 		(unit 1)
 		(body_style 1)
 		(exclude_from_sim no)
-		(in_bom yes)
+		(in_bom no)
 		(on_board yes)
-		(in_pos_files yes)
+		(in_pos_files no)
 		(dnp no)
+		(fields_autoplaced yes)
 		(property "Reference" "TP6"
-			(at 249.174 20.574 0)
+			(at 252.73 19.05 0)
 			(show_name no)
 			(do_not_autoplace no)
@@
 					(size 1.27 1.27)
 				)
-				(justify left)
 			)
 		)
 		(property "Value" "TestPoint"
-			(at 247.65 22.098 0)
+			(at 252.73 21.59 0)
 			(show_name no)
 			(do_not_autoplace no)
@@
 					(size 1.27 1.27)
 				)
-				(justify left)
 			)
 		)
-		(property "Footprint" "TestPoint:TestPoint_Pad_D1.0mm"
-			(at 257.81 29.21 0)
+		(property "Footprint" "Testpoints_Kampi:TestPoint_Pad_D1.0mm"
+			(at 257.81 27.94 0)
 			(hide yes)
 			(show_name no)
@@
 		)
 		(property "Datasheet" ""
-			(at 257.81 29.21 0)
+			(at 257.81 27.94 0)
 			(hide yes)
 			(show_name no)
@@
 		)
 		(property "Description" "test point"
-			(at 252.73 29.21 0)
+			(at 252.73 27.94 0)
+			(hide yes)
+			(show_name no)
+			(do_not_autoplace no)
+			(effects
+				(font
+					(size 1.27 1.27)
+				)
+			)
+		)
+		(property "manf" ""
+			(at 252.73 27.94 0)
+			(hide yes)
+			(show_name no)
+			(do_not_autoplace no)
+			(effects
+				(font
+					(size 1.27 1.27)
+				)
+			)
+		)
+		(property "manf#" ""
+			(at 252.73 27.94 0)
+			(hide yes)
+			(show_name no)
+			(do_not_autoplace no)
+			(effects
+				(font
+					(size 1.27 1.27)
+				)
+			)
+		)
+		(property "mouser#" ""
+			(at 252.73 27.94 0)
+			(hide yes)
+			(show_name no)
+			(do_not_autoplace no)
+			(effects
+				(font
+					(size 1.27 1.27)
+				)
+			)
+		)
+		(property "Config" ""
+			(at 252.73 27.94 0)
 			(hide yes)
 			(show_name no)
@@
 	(symbol
 		(lib_id "Connector:TestPoint")
-		(at 242.57 101.6 0)
+		(at 242.57 100.33 0)
 		(unit 1)
 		(body_style 1)
 		(exclude_from_sim no)
-		(in_bom yes)
+		(in_bom no)
 		(on_board yes)
-		(in_pos_files yes)
+		(in_pos_files no)
 		(dnp no)
+		(fields_autoplaced yes)
 		(property "Reference" "TP5"
-			(at 239.014 92.964 0)
+			(at 242.57 91.44 0)
 			(show_name no)
 			(do_not_autoplace no)
@@
 					(size 1.27 1.27)
 				)
-				(justify left)
 			)
 		)
 		(property "Value" "TestPoint"
-			(at 237.49 94.488 0)
+			(at 242.57 93.98 0)
 			(show_name no)
 			(do_not_autoplace no)
@@
 					(size 1.27 1.27)
 				)
-				(justify left)
 			)
 		)
-		(property "Footprint" "TestPoint:TestPoint_Pad_D1.0mm"
-			(at 247.65 101.6 0)
+		(property "Footprint" "Testpoints_Kampi:TestPoint_Pad_D1.0mm"
+			(at 247.65 100.33 0)
 			(hide yes)
 			(show_name no)
@@
 		)
 		(property "Datasheet" ""
-			(at 247.65 101.6 0)
+			(at 247.65 100.33 0)
 			(hide yes)
 			(show_name no)
@@
 		)
 		(property "Description" "test point"
-			(at 242.57 101.6 0)
+			(at 242.57 100.33 0)
+			(hide yes)
+			(show_name no)
+			(do_not_autoplace no)
+			(effects
+				(font
+					(size 1.27 1.27)
+				)
+			)
+		)
+		(property "manf" ""
+			(at 242.57 100.33 0)
+			(hide yes)
+			(show_name no)
+			(do_not_autoplace no)
+			(effects
+				(font
+					(size 1.27 1.27)
+				)
+			)
+		)
+		(property "manf#" ""
+			(at 242.57 100.33 0)
+			(hide yes)
+			(show_name no)
+			(do_not_autoplace no)
+			(effects
+				(font
+					(size 1.27 1.27)
+				)
+			)
+		)
+		(property "mouser#" ""
+			(at 242.57 100.33 0)
+			(hide yes)
+			(show_name no)
+			(do_not_autoplace no)
+			(effects
+				(font
+					(size 1.27 1.27)
+				)
+			)
+		)
+		(property "Config" ""
+			(at 242.57 100.33 0)
 			(hide yes)
 			(show_name no)
@@
 	(symbol
 		(lib_id "Connector:TestPoint")
-		(at 242.57 83.82 0)
+		(at 242.57 82.55 0)
 		(unit 1)
 		(body_style 1)
 		(exclude_from_sim no)
-		(in_bom yes)
+		(in_bom no)
 		(on_board yes)
-		(in_pos_files yes)
+		(in_pos_files no)
 		(dnp no)
+		(fields_autoplaced yes)
 		(property "Reference" "TP4"
-			(at 239.014 75.184 0)
+			(at 242.57 73.66 0)
 			(show_name no)
 			(do_not_autoplace no)
@@
 					(size 1.27 1.27)
 				)
-				(justify left)
 			)
 		)
 		(property "Value" "TestPoint"
-			(at 237.49 76.708 0)
+			(at 242.57 76.2 0)
 			(show_name no)
 			(do_not_autoplace no)
@@
 					(size 1.27 1.27)
 				)
-				(justify left)
 			)
 		)
-		(property "Footprint" "TestPoint:TestPoint_Pad_D1.0mm"
-			(at 247.65 83.82 0)
+		(property "Footprint" "Testpoints_Kampi:TestPoint_Pad_D1.0mm"
+			(at 247.65 82.55 0)
 			(hide yes)
 			(show_name no)
@@
 		)
 		(property "Datasheet" ""
-			(at 247.65 83.82 0)
+			(at 247.65 82.55 0)
 			(hide yes)
 			(show_name no)
@@
 		)
 		(property "Description" "test point"
-			(at 242.57 83.82 0)
+			(at 242.57 82.55 0)
+			(hide yes)
+			(show_name no)
+			(do_not_autoplace no)
+			(effects
+				(font
+					(size 1.27 1.27)
+				)
+			)
+		)
+		(property "manf" ""
+			(at 242.57 82.55 0)
+			(hide yes)
+			(show_name no)
+			(do_not_autoplace no)
+			(effects
+				(font
+					(size 1.27 1.27)
+				)
+			)
+		)
+		(property "manf#" ""
+			(at 242.57 82.55 0)
+			(hide yes)
+			(show_name no)
+			(do_not_autoplace no)
+			(effects
+				(font
+					(size 1.27 1.27)
+				)
+			)
+		)
+		(property "mouser#" ""
+			(at 242.57 82.55 0)
+			(hide yes)
+			(show_name no)
+			(do_not_autoplace no)
+			(effects
+				(font
+					(size 1.27 1.27)
+				)
+			)
+		)
+		(property "Config" ""
+			(at 242.57 82.55 0)
 			(hide yes)
 			(show_name no)
