File: watch/ZSWatch-Watch.kicad_pcb (KiCad board)
At the start: 4 copper layers, 41 x 37.5 mm, 64 parts, among them IC401 nPM1300-QEXX, IC501 APDS-9306-065, IC502 BMI270, IC503 LIS2MDLTR, IC504 BMP581, IC505 DRV2603RUNT, IC506 PCA9306JK, IC507 RV-8263-C8, IC601 FAN5622SX, IC602 USBLC6-2P6, IC603 MX25U51245GZ4I00, IC604 NTS0104GU12, M601 NORA-B106, X402 Battery, X509 Motor, X603 Device, X608 Display, X701 MB1, X702 MB2

Commit message: Update outputs (release)
Other:
- board text added: "0.035mm (1.00oz)"
- board text added: "0.43mm"
- board text added: "Inner1"
- board text added: "Total thickness: 0.982mm"
- board text removed: "0.035mm (1oz)"
- board text removed: "1.03mm"
- board text removed: "Inner1 (GND)"
- board text removed: "Total thickness: 1.582mm"
